File: platine/AutomatedBlinds/AutomatedBlinds.kicad_pcb (KiCad board)
At the start: 2 copper layers, 72.5 x 47 mm, 12 parts, among them J2 Conn_01x03_Male, J4 Conn_01x07_Male, SW1 SW_Push, SW2 SW_Push

Commit message: minor
Routing:
- net Net-(A1-D11): track 0.00 -> 4.80 mm
Other:
- board text added: "AutoBlinds v2.1"
Changed lines of the file:
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@@
 		(layer "Edge.Cuts")
+	)
+	(gr_text "AutoBlinds v2.1"
+		(at 180.5 73 0)
+		(layer "B.Cu" knockout)
+		(effects
+			(font
+				(size 1.5 1.5)
+				(thickness 0.3)
+				(bold yes)
+			)
+			(justify left bottom mirror)
+		)
+	)
+	(gr_text "6V"
+		(at 124.96 112 90)
+		(layer "B.Cu" knockout)
+		(effects
+			(font
+				(size 1 1)
+				(thickness 0.15)
+			)
+			(justify left bottom)
+		)
 	)
 	(gr_text "SDA"
@@
 		)
 	)
-	(gr_text "6V"
-		(at 124.96 106 90)
-		(layer "F.SilkS")
-		(effects
-			(font
-				(size 1 1)
-				(thickness 0.15)
-			)
-			(justify left bottom)
-		)
-	)
 	(segment
 		(start 129.34 106.915445)
@@
 	)
 	(segment
+		(start 140.74 108)
+		(end 143.26 105.48)
+		(width 0.2)
+		(layer "B.Cu")
+		(net 24)
+	)
+	(segment
+		(start 139.5 108)
+		(end 140.74 108)
+		(width 0.2)
+		(layer "B.Cu")
+		(net 24)
+	)
+	(segment
